Commit message: slam funcionando

File: src/my_robot_description/urdf/imu.xacro (robot description, xacro)
@@ -9,5 +9,5 @@
                 <box size="${imu_length} ${imu_width} ${imu_height}" />
             </geometry>
-            <material name="green" />
+            <material name="grey" />
         </visual>
         <collision>

File: src/my_robot_description/urdf/mobile_base.xacro (robot description, xacro)
@@ -1,6 +1,6 @@
 <?xml version="1.0"?>
 <robot xmlns:xacro="http://www.ros.org/wiki/xacro">
-    <xacro:property name="base_length" value="0.6" />
-    <xacro:property name="base_width" value="0.4" />
+    <xacro:property name="base_length" value="0.35" />
+    <xacro:property name="base_width" value="0.25" />
     <xacro:property name="base_height" value="0.2" />
     <xacro:property name="wheel_radius" value="0.1" />

File: src/my_robot_description/urdf/nav_lidar.xacro (robot description, xacro)
@@ -3,9 +3,9 @@
     <xacro:property name="lidar_radius" value="0.035" />
     <xacro:property name="lidar_height" value="0.042" />
-    <xacro:property name="two_d_lidar_sample_size" value="120"/>
-    <xacro:property name="two_d_lidar_min_angle" value="-3.14159"/>
-    <xacro:property name="two_d_lidar_max_angle" value="3.14159"/>
-    <xacro:property name="two_d_lidar_min_range" value="0.16"/>
-    <xacro:property name="two_d_lidar_max_range" value="8"/>
+    <xacro:property name="two_d_lidar_sample_size" value="361"/>
+    <xacro:property name="two_d_lidar_min_angle" value="-180"/>
+    <xacro:property name="two_d_lidar_max_angle" value="180"/>
+    <xacro:property name="two_d_lidar_min_range" value="0.12"/>
+    <xacro:property name="two_d_lidar_max_range" value="3.5"/>
     <link name="lidar_link">
         <visual>
@@ -13,5 +13,5 @@
                 <cylinder radius="${lidar_radius}" length="${lidar_height}" />
             </geometry>
-            <material name="black" />
+            <material name="grey" />
         </visual>
         <collision>
@@ -54,11 +54,11 @@
                     <type>gaussian</type>
                     <mean>0.0</mean>
-                    <stddev>0.0</stddev>
+                    <stddev>0.01</stddev>
                 </noise>
             </ray>
             <plugin name="gazebo_ros_laser" filename="libgazebo_ros_ray_sensor.so">
                 <ros>
-                    <namespace>/ray</namespace>
-                    <remapping>~/out:=laserscan</remapping>
+                    <output>screen</output>
+                    <remapping>~/out:=/scan</remapping>
                 </ros>
                 <output_type>sensor_msgs/LaserScan</output_type>

File: src/my_robot_description/urdf/nav_mobile_base_gazebo.xacro (robot description, xacro)
@@ -42,7 +42,7 @@
             <odometry_source>1</odometry_source>
             <!-- Change the ROS topic we will publish the odometry data to -->
-            <ros>
+            <!-- <ros>
             <remapping>odom:=wheel/odometry</remapping>
-            </ros>
+            </ros> -->
         </plugin>
     </gazebo>
